Commit message: Working lab trials

File: pruning_bt/srdf/system_macro.srdf.xacro (robot description, xacro)
@@ -42,39 +42,42 @@
     <!--VIRTUAL JOINT - Purpose - this element defines a virtual joint between a robot link and an external frame of reference (considered fixed with respect to the robot)-->
     <!--DISABLE COLLISIONS - By default it is assumed that any link of the robot could potentially come into collision with any other link in the robot. This tag disables collision checking between a specified pair of links. -->
-    <disable_collisions link1="${prefix}base_link" link2="${prefix}base_link_inertia" reason="Adjacent" />
-    <disable_collisions link1="${prefix}base_link_inertia" link2="${prefix}shoulder_link" reason="Adjacent" />
-    <disable_collisions link1="${prefix}tool0" link2="${prefix}wrist_1_link" reason="Never" />
-    <disable_collisions link1="${prefix}tool0" link2="${prefix}wrist_2_link" reason="Never" />
-    <disable_collisions link1="${prefix}tool0" link2="${prefix}wrist_3_link" reason="Adjacent" />
-    <disable_collisions link1="${prefix}forearm_link" link2="${prefix}upper_arm_link" reason="Adjacent" />
-    <disable_collisions link1="${prefix}forearm_link" link2="${prefix}wrist_1_link" reason="Adjacent" />
-    <disable_collisions link1="${prefix}shoulder_link" link2="${prefix}upper_arm_link" reason="Adjacent" />
-    <disable_collisions link1="${prefix}wrist_1_link" link2="${prefix}wrist_2_link" reason="Adjacent" />
-    <disable_collisions link1="${prefix}wrist_1_link" link2="${prefix}wrist_3_link" reason="Never" />
-    <disable_collisions link1="${prefix}wrist_2_link" link2="${prefix}wrist_3_link" reason="Adjacent" />
-    <disable_collisions link1="${prefix}wrist_3_link" link2="${prefix}dovetail_male_mount__base" reason="Adjacent" />
-    <disable_collisions link1="${prefix}wrist_3_link" link2="${prefix}rotation_correction_plate__body" reason="Adjacent" />
-    <disable_collisions link1="${prefix}dovetail_male_mount__base" link2="${prefix}rotation_correction_plate__base" reason="Adjacent" />
-    <disable_collisions link1="${prefix}dovetail_male_mount__base" link2="${prefix}rotation_correction_plate__body" reason="Adjacent" />
-    <disable_collisions link1="${prefix}rotation_correction_plate__base" link2="${prefix}rotation_correction_plate__body" reason="Adjacent" />
-    <disable_collisions link1="${prefix}rotation_correction_plate__body" link2="${prefix}dovetail_male_mount__base" reason="Adjacent" />
-        <!-- Male to Male Dovetail Part Collisions -->
-    <disable_collisions link1="${prefix}dovetail_male_mount__base" link2="${prefix}dovetail_male_mount__body" reason="Adjacent" />
-    <disable_collisions link1="${prefix}dovetail_male_mount__base" link2="${prefix}dovetail_male_mount__tool0" reason="Adjacent" />
-    <disable_collisions link1="${prefix}dovetail_male_mount__body" link2="${prefix}dovetail_male_mount__tool0" reason="Adjacent" />
-    <!-- Female to Female Dovetail Part Collisions -->
-    <disable_collisions link1="${prefix}dovetail_female_mount__base" link2="${prefix}dovetail_female_mount__body" reason="Adjacent" />
-    <disable_collisions link1="${prefix}dovetail_female_mount__base" link2="${prefix}dovetail_female_mount__tool0" reason="Adjacent" />
-    <disable_collisions link1="${prefix}dovetail_female_mount__body" link2="${prefix}dovetail_female_mount__tool0" reason="Adjacent" />
-    <!-- Male to Female Dovetail Part Collisions -->
-    <disable_collisions link1="${prefix}dovetail_male_mount__base" link2="${prefix}dovetail_female_mount__base" reason="Adjacent" />
-    <disable_collisions link1="${prefix}dovetail_male_mount__base" link2="${prefix}dovetail_female_mount__body" reason="Adjacent" />
-    <disable_collisions link1="${prefix}dovetail_male_mount__base" link2="${prefix}dovetail_female_mount__tool0" reason="Adjacent" />
-    <disable_collisions link1="${prefix}dovetail_male_mount__body" link2="${prefix}dovetail_female_mount__base" reason="Adjacent" />
-    <disable_collisions link1="${prefix}dovetail_male_mount__body" link2="${prefix}dovetail_female_mount__body" reason="Adjacent" />
-    <disable_collisions link1="${prefix}dovetail_male_mount__body" link2="${prefix}dovetail_female_mount__tool0" reason="Adjacent" />
-    <disable_collisions link1="${prefix}dovetail_male_mount__tool0" link2="${prefix}dovetail_female_mount__base" reason="Adjacent" />
-    <disable_collisions link1="${prefix}dovetail_male_mount__tool0" link2="${prefix}dovetail_female_mount__body" reason="Adjacent" />
-    <disable_collisions link1="${prefix}dovetail_male_mount__tool0" link2="${prefix}dovetail_female_mount__tool0" reason="Adjacent" />
+    <disable_collisions link1="amiga__body" link2="base_link_inertia" reason="Never" />
+  <disable_collisions link1="amiga__body" link2="base_link" reason="Never" />
+  <disable_collisions link1="amiga__tool0" link2="base_link_inertia" reason="Never" />
+  <disable_collisions link1="amiga__tool0" link2="base_link" reason="Never" />
+  <disable_collisions link1="base_link" link2="base_link_inertia" reason="Adjacent" />
+  <disable_collisions link1="base_link_inertia" link2="shoulder_link" reason="Adjacent" />
+  <disable_collisions link1="tool0" link2="wrist_1_link" reason="Never" />
+  <disable_collisions link1="tool0" link2="wrist_2_link" reason="Never" />
+  <disable_collisions link1="tool0" link2="wrist_3_link" reason="Adjacent" />
+  <disable_collisions link1="forearm_link" link2="upper_arm_link" reason="Adjacent" />
+  <disable_collisions link1="forearm_link" link2="wrist_1_link" reason="Adjacent" />
+  <disable_collisions link1="shoulder_link" link2="upper_arm_link" reason="Adjacent" />
+  <disable_collisions link1="wrist_1_link" link2="wrist_2_link" reason="Adjacent" />
+  <disable_collisions link1="wrist_1_link" link2="wrist_3_link" reason="Never" />
+  <disable_collisions link1="wrist_2_link" link2="wrist_3_link" reason="Adjacent" />
+  <disable_collisions link1="rotation_correction_plate__base" link2="tool0" reason="Adjacent" />
+  <disable_collisions link1="rotation_correction_plate__base" link2="wrist_3_link" reason="Never" />
+  <disable_collisions link1="rotation_correction_plate__body" link2="tool0" reason="Adjacent" />
+  <disable_collisions link1="rotation_correction_plate__body" link2="wrist_3_link" reason="Never" />
+  <disable_collisions link1="rotation_correction_plate__body" link2="dovetail_male_mount__base" reason="Adjacent" />
+  <disable_collisions link1="rotation_correction_plate__body" link2="dovetail_male_mount__body" reason="Never" />
+  <disable_collisions link1="rotation_correction_plate__tool0" link2="dovetail_male_mount__base" reason="Adjacent" />
+  <disable_collisions link1="rotation_correction_plate__tool0" link2="dovetail_male_mount__body" reason="Never" />
+  <disable_collisions link1="dovetail_male_mount__base" link2="tool0" reason="Never" />
+  <disable_collisions link1="dovetail_male_mount__base" link2="dovetail_male_mount__body" reason="Never" />
+  <disable_collisions link1="dovetail_male_mount__base" link2="dovetail_male_mount__tool0" reason="Never" />
+  <disable_collisions link1="dovetail_male_mount__body" link2="tool0" reason="Never" />
+  <disable_collisions link1="dovetail_male_mount__body" link2="wrist_3_link" reason="Never" />
+  <disable_collisions link1="dovetail_female_mount__base" link2="dovetail_male_mount__tool0" reason="Adjacent" />
+  <disable_collisions link1="dovetail_female_mount__base" link2="dovetail_male_mount__body" reason="Adjacent" />
+  <disable_collisions link1="dovetail_female_mount__body" link2="dovetail_male_mount__body" reason="Never" />
+  <disable_collisions link1="dovetail_female_mount__body" link2="dovetail_male_mount__tool0" reason="Never" />
+  <disable_collisions link1="dovetail_female_mount__body" link2="wrist_3_link" reason="Never" />
+  <disable_collisions link1="dovetail_female_mount__body" link2="tool0" reason="Never" />
+  <disable_collisions link1="mock_pruner__base" link2="dovetail_female_mount__tool0" reason="Adjacent" />
+  <disable_collisions link1="mock_pruner__base" link2="dovetail_female_mount__body" reason="Never" />
+  <disable_collisions link1="mock_pruner__base" link2="dovetail_male_mount__body" reason="Never" />
+  <disable_collisions link1="mock_pruner__base" link2="dovetail_male_mount__tool0" reason="Never" />
     <!-- Cutter Part Collisions -->
     <disable_collisions link1="${prefix}dovetail_female_mount__body" link2="${prefix}mock_pruner__base" reason="Adjacent" />
@@ -85,40 +88,4 @@
     <disable_collisions link1="${prefix}mock_pruner__mouth" link2="${prefix}mock_pruner__base" reason="Adjacent" />
     <disable_collisions link1="${prefix}mock_pruner__mouth" link2="${prefix}mock_pruner__mouth_base" reason="Adjacent" />
-    <disable_collisions link1="cart__tool0" link2="ur5e__base_link" reason="Never" />
-    <disable_collisions link1="${prefix}base_link" link2="${prefix}base_link_inertia" reason="Adjacent" />
-    <disable_collisions link1="${prefix}base_link_inertia" link2="${prefix}shoulder_link" reason="Adjacent" />
-    <disable_collisions link1="${prefix}tool0" link2="${prefix}wrist_1_link" reason="Never" />
-    <disable_collisions link1="${prefix}tool0" link2="${prefix}wrist_2_link" reason="Never" />
-    <disable_collisions link1="${prefix}tool0" link2="${prefix}wrist_3_link" reason="Adjacent" />
-    <disable_collisions link1="${prefix}forearm_link" link2="${prefix}upper_arm_link" reason="Adjacent" />
-    <disable_collisions link1="${prefix}forearm_link" link2="${prefix}wrist_1_link" reason="Adjacent" />
-    <disable_collisions link1="${prefix}shoulder_link" link2="${prefix}upper_arm_link" reason="Adjacent" />
-    <disable_collisions link1="${prefix}wrist_1_link" link2="${prefix}wrist_2_link" reason="Adjacent" />
-    <disable_collisions link1="${prefix}wrist_1_link" link2="${prefix}wrist_3_link" reason="Never" />
-    <disable_collisions link1="${prefix}wrist_2_link" link2="${prefix}wrist_3_link" reason="Adjacent" />
-    <!-- TODO Dynamically configure. Can probably be done with just the "body" links? Or maybe virtual links here. -->
-    <disable_collisions link1="rotation_correction_plate__base" link2="${prefix}tool0" reason="Adjacent" />
-    <disable_collisions link1="rotation_correction_plate__base" link2="${prefix}wrist_3_link" reason="Never" />
-    <disable_collisions link1="rotation_correction_plate__body" link2="${prefix}tool0" reason="Adjacent" />
-    <disable_collisions link1="rotation_correction_plate__body" link2="${prefix}wrist_3_link" reason="Never" />
-    <disable_collisions link1="rotation_correction_plate__body" link2="dovetail_male_mount__base" reason="Adjacent" />
-    <disable_collisions link1="rotation_correction_plate__body" link2="dovetail_male_mount__body" reason="Never" />
-    <disable_collisions link1="rotation_correction_plate__tool0" link2="dovetail_male_mount__base" reason="Adjacent" />
-    <disable_collisions link1="rotation_correction_plate__tool0" link2="dovetail_male_mount__body" reason="Never" />
-    <disable_collisions link1="dovetail_male_mount__base" link2="${prefix}tool0" reason="Never" />
-    <disable_collisions link1="dovetail_male_mount__base" link2="dovetail_male_mount__body" reason="Never" />
-    <disable_collisions link1="dovetail_male_mount__base" link2="dovetail_male_mount__tool0" reason="Never" />
-    <disable_collisions link1="dovetail_male_mount__body" link2="${prefix}tool0" reason="Never"/>
-    <disable_collisions link1="dovetail_male_mount__body" link2="${prefix}wrist_3_link" reason="Never"/>
-    <disable_collisions link1="dovetail_female_mount__base" link2="dovetail_male_mount__tool0" reason="Adjacent" />
-    <disable_collisions link1="dovetail_female_mount__base" link2="dovetail_male_mount__body" reason="Adjacent" />
-    <disable_collisions link1="dovetail_female_mount__body" link2="dovetail_male_mount__body" reason="Never" />
-    <disable_collisions link1="dovetail_female_mount__body" link2="dovetail_male_mount__tool0" reason="Never" />
-    <disable_collisions link1="dovetail_female_mount__body" link2="${prefix}wrist_3_link" reason="Never"/>
-    <disable_collisions link1="dovetail_female_mount__body" link2="${prefix}tool0" reason="Never"/>
-    <disable_collisions link1="mock_pruner__base" link2="dovetail_female_mount__tool0" reason="Adjacent" />
-    <disable_collisions link1="mock_pruner__base" link2="dovetail_female_mount__body" reason="Never" />
-    <disable_collisions link1="mock_pruner__base" link2="dovetail_male_mount__body" reason="Never" />
-    <disable_collisions link1="mock_pruner__base" link2="dovetail_male_mount__tool0" reason="Never" />
 <!--
     <disable_collisions link1="${prefix}dovetail_male_mount__base" link2="${prefix}dovetail_male_mount__body" reason="Adjacent" />

File: pruning_bt/urdf/ur5_with_pruner.urdf.xacro (robot description, xacro)
@@ -51,9 +51,58 @@
    <!-- create link fixed to the "world" -->
    <link name="world" />
+   <link name="amiga__base" />
+    <link name="amiga__body">
+      <visual>
+        <origin rpy="0.0 0.0 0.0" xyz="0.0 0.0 0.0" />
+        <geometry>
+          <mesh filename="package://pruning_bt/meshes/base_mounts/farm-ng/amiga/frame_on_amiga_v2_simplified.stl" />
+        </geometry>
+        <material name="LightLightGrey" />
+      </visual>
+      <collision>
+        <origin rpy="0.0 0.0 0.0" xyz="0.0 0.0 0.499053035" />
+        <geometry>
+          <box size="1.132 0.8 0.99810607" />
+        </geometry>
+      </collision>
+      <collision>
+        <origin rpy="0.0 0.0 0.0" xyz="0.0 -0.12 0.99810607" />
+        <geometry>
+          <box size="1.132 0.6 0.2" />
+        </geometry>
+      </collision>
+      <collision>
+        <origin rpy="0.0 0.0 0.0" xyz="0.44099999999999995 0.08333333333333333 1.19810607" />
+        <geometry>
+          <box size="0.25 0.25 0.25" />
+        </geometry>
+      </collision>
+      <inertial>
+        <origin rpy="0 0 0" xyz="0.0 0.0 0.0" />
+        <mass value="40.0" />
+        <inertia ixx="5.454052423236149" ixy="0.0" ixz="0.0" iyy="7.592132423236148" iyz="0.0" izz="6.404746666666665" />
+      </inertial>
+    </link>
+    <link name="amiga__tool0" />
+    <joint name="world--amiga__base" type="fixed">
+      <origin rpy="0 0 3.14159265359" xyz="0 0 0" />
+      <parent link="world" />
+      <child link="amiga__base" />
+    </joint>
+    <joint name="amiga__base--amiga__body" type="fixed">
+      <origin rpy="0 0 0" xyz="0 0 0" />
+      <parent link="amiga__base" />
+      <child link="amiga__body" />
+    </joint>
+    <joint name="amiga__body--amiga__tool0" type="fixed">
+      <origin rpy="0.0 0.0 -3.9269908169872414" xyz="-0.225 0.323256 0.99810607" />
+      <parent link="amiga__body" />
+      <child link="amiga__tool0" />
+    </joint>
    <!-- arm -->
    <xacro:ur_robot
      name="$(arg name)"
      tf_prefix="$(arg tf_prefix)"
-     parent="world"
+     parent="amiga__tool0"
      joint_limits_parameters_file="$(arg joint_limit_params)"
      kinematics_parameters_file="$(arg kinematics_params)"
@@ -91,4 +140,10 @@
      <origin xyz="0 0 0" rpy="0 0 0" />          <!-- position robot in the world -->
    </xacro:ur_robot>
+<!--
+  <joint name="base_joint" type="fixed">
+    <origin rpy="0 0 0" xyz="0 0 0" />
+    <parent link="amiga__tool0" />
+    <child link="base_link" />
+  </joint> -->
    <xacro:if value="$(arg sim_gazebo)">
     <!-- Gazebo plugins -->
@@ -118,5 +173,5 @@
       <origin rpy="0 0 0" xyz="0 0 0" />
       <geometry>
-        <mesh filename="package://pruning_bt/meshes/RotationCorrectionPlate.STL" />
+        <mesh filename="package://pruning_bt/meshes/end_effectors/rotation_correction_plate/RotationCorrectionPlate.STL" />
       </geometry>
     </visual>
@@ -124,5 +179,5 @@
       <origin rpy="0 0 0" xyz="0 0 0" />
       <geometry>
-        <mesh filename="package://pruning_bt/meshes/RotationCorrectionPlate.STL" />
+        <mesh filename="package://pruning_bt/meshes/end_effectors/rotation_correction_plate/RotationCorrectionPlate.STL" />
       </geometry>
     </collision>
@@ -158,5 +213,5 @@
       <origin rpy="0 0 0" xyz="0 0 0" />
       <geometry>
-        <mesh filename="package://pruning_bt/meshes/DovetailMale.STL" />
+        <mesh filename="package://pruning_bt/meshes/end_effectors/dovetail/DovetailMale.STL" />
       </geometry>
     </visual>
@@ -164,5 +219,5 @@
       <origin rpy="0 0 0" xyz="0 0 0" />
       <geometry>
-        <mesh filename="package://pruning_bt/meshes/DovetailMale.STL" />
+        <mesh filename="package://pruning_bt/meshes/end_effectors/dovetail/DovetailMale.STL" />
       </geometry>
     </collision>
@@ -198,5 +253,5 @@
       <origin rpy="0 0 0" xyz="0 0 0" />
       <geometry>
-        <mesh filename="package://pruning_bt/meshes/DovetailFemale.STL" />
+        <mesh filename="package://pruning_bt/meshes/end_effectors/dovetail/DovetailFemale.STL" />
       </geometry>
     </visual>
@@ -204,5 +259,5 @@
       <origin rpy="0 0 0" xyz="0 0 0" />
       <geometry>
-        <mesh filename="package://pruning_bt/meshes/DovetailFemale.STL" />
+        <mesh filename="package://pruning_bt/meshes/end_effectors/dovetail/DovetailFemale.STL" />
       </geometry>
     </collision>
@@ -236,5 +291,5 @@
       <origin rpy="0 0 0" xyz="0 0 0" />
       <geometry>
-        <mesh filename="package://pruning_bt/meshes/MockPrunerNoToF.STL" />
+        <mesh filename="package://pruning_bt/meshes/end_effectors/mock_pruner/MockPrunerNoToF.STL" />
       </geometry>
     </visual>
@@ -242,5 +297,5 @@
       <origin rpy="0 0 0" xyz="0 0 0" />
       <geometry>
-        <mesh filename="package://pruning_bt/meshes/MockPrunerNoToF.STL" />
+        <mesh filename="package://pruning_bt/meshes/end_effectors/mock_pruner/MockPrunerNoToF.STL" />
       </geometry>
     </collision>
